File: mcu.kicad_sch (KiCad schematic)
At the start: 19 parts, among them J2 Conn_01x05, J3 Conn_01x02, U1 TPS73233DBVR, U3 STM32G070KBT6

Commit message: Add CI script (#2)
* Renamed main files to SCAN2000

* Add CI

* Bump version to 1.1.1

* Remove the BOM as this is now generated content

* Reworked Readme
Parts:
- J2: PN 69190-405HLF -> 69190-405HLF
Changed lines of the file:
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@@
 			)
 		)
-		(property "PN" " 69190-405HLF"
+		(property "PN" "69190-405HLF"
 			(at 240.03 40.64 0)
 			(effects
