File: relays.kicad_sch (KiCad schematic)
At the start: 0 parts

Commit message: Updated BOM
Other:
- note added: "A note on the Relays: With SSRs, there is always a compromise between on-state resistance and leakage current. This project is aimed to replace the majority of use cases of a replay card. - The K2002 manual states the following requirements for the OHMS range: The lead resistance on the 20 Ω range must be < 10 Ω on the LO side. - The DMM6500 says "5 Ω per lead for 1 Ω range". The relays used have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"
Changed lines of the file:
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@@
     (stroke (width 0) (type default) (color 0 0 0 0))
+  )
+  (text "A note on the Relays:\nWith SSRs, there is always a compromise between on-state resistance and leakage current.\nThis project is aimed to replace the majority of use cases of a replay card.\n- The K2002 manual states the following requirements for the OHMS range:\n   The lead resistance on the 20 Ω range must be < 10 Ω on the LO side.\n- The DMM6500 says \"5 Ω per lead for 1 Ω range\".\n\nThe relays used have a maximum on-state resistance of 2 Ω. Well below that requirement.\nThey are also rated for 700 mA and 200 V.\nThe downside is the leakage current of < 1 µA. The typical value is 40 nA, but there is no guarantee.\n\nThe original 2000-SCAN card is rated for 110V, 1A, < 1 Ω contact resistance and\na maximum contact potential of 1 µV, so this replacement is very close to the original 2000-SCAN card."
+    (at 146.05 52.07 0)
+    (effects (font (size 1.27 1.27)) (justify left bottom))
   )
   (hierarchical_label "CH2" (shape input) (at 76.2 43.18 180)
