File: fpga.kicad_sch (KiCad schematic)
At the start: 39 parts, among them J5 Conn_02x05_Odd_Even, U1 ASDAIG-16.000MHZ-C-S-T, U25 ICE40HX1K-TQ144, U48 W25Q16JVS, U49 TLV71312PQDBVRQ1, U50 LDK130M33RY

Commit message: Updated BOM properties
Parts:
- JP2: DNP (none) -> 1; now left out of the parts list
- TP5: now not fitted
Changed lines of the file:
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@@
 		(in_bom yes)
 		(on_board yes)
-		(dnp no)
+		(dnp yes)
 		(property "Reference" "TP5"
 			(at 254 15.24 0)
@@
 		(unit 1)
 		(exclude_from_sim no)
-		(in_bom yes)
+		(in_bom no)
 		(on_board yes)
 		(dnp no)
@@
 			(at 231.14 127 0)
 			(effects
+				(font
+					(size 1.27 1.27)
+				)
+				(hide yes)
+			)
+		)
+		(property "DNP" "1"
+			(at 231.14 127 0)
+			(effects
